File: avoccado-avr-pcb-nora/panel/avoccado-nora-panel.brd (EAGLE design)
At the start: 50 x 50 mm, 51 parts, among them Q1 16MHz, Q2 FET, U2 MCP73831

Commit message: panelized nora to 50x50mm²
Parts:
- added LOGO2: OSHW-LOGOS, SparkFun-Aesthetics:OSHW-LOGO-S
Routing:
- net D2: track 38.6 -> 19.6 mm, vias 1 -> 2
- net 3.3V: track 77.5 -> 83.4 mm
- net D4: track 23.7 -> 26.5 mm
- net GND: track 124.5 -> 126.8 mm
- net A4: track 1.48 -> 3.38 mm
- net A5: track 1.72 -> 2.99 mm
Other:
- board size 50 x 50 mm -> 23.9 x 23.4 mm
- board text added: "AVOCCADO NORA 1"
- board text removed: "ATMEGA328"
- board text removed: "AVOCCADO YOLANDI"
