File: avoccado-avr-pcb-nora/avoccado-nora-test-jig/avoccado-nora-test-jig.sch (EAGLE design)
At the start: 29 parts, among them J1 AVR_SPI_PROG2PTH2

Commit message: switch layer for ICSP 2x5 header to bottom
Parts:
- removed J1: AVR_SPI_PROG2PTH2, SparkFun-Connectors:AVR_SPI_PROG2PTH2
- removed JP19, JP20, JP21, JP22, JP23, JP24, JP25, JP26, TP2: M01NOSILK-KIT, SparkFun-Connectors:M01NOSILK-KIT
- removed JP4, JP5: M021X02_NO_SILK, SparkFun-Connectors:M021X02_NO_SILK
- added R1: 0, SparkFun-Passives:RESISTOR1206
- added SJ1: JUMPER-PAD-2-NC_BY_TRACE, SparkFun-Passives:JUMPER-PAD-2-NC_BY_TRACE
- added SJ2: JUMPER-PAD-2-NO, SparkFun-Passives:JUMPER-PAD-2-NO
Connections:
- removed net A0: JP19.1
- removed net A1: JP20.1
- removed net A2: JP21.1
- removed net A3: JP22.1
- removed net A4: JP5.2
- removed net A5: JP5.1
- removed net D2: TP2.1
- removed net VBAT: JP24.1
- removed net VIBR: JP23.1
- new net MISO1: ICSP.9, R1.2
- new net VTG: ICSP.2, SJ1.2, SJ2.2
- net 3.3V: now also SJ1.1; no longer ICSP.2, JP4.1
- net 5V: now also SJ2.1
- net GND: no longer JP25.1, JP26.1, JP4.2
- net MISO: now also R1.1; no longer ICSP.9
Other:
- note removed: "MPU6050 minimal header I2C"
- note removed: "NRF24L01+ board header SPI (IRQ at A7)"
- note removed: "UART/Serial interface (unrouted)"
- moved on the sheet: JP10, JP11, JP17, JP18, JP3, JP6, JP8, JP9, TP1, TP6, TP7, TP8

Commit message: ditch DTR line at ICSP header
Connections:
- net DTR: no longer ICSP.8
Changed lines of the file:
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@@
 </segment>
 <segment>
-<wire x1="35.56" y1="17.78" x2="43.18" y2="17.78" width="0.1524" layer="91"/>
-<pinref part="ICSP" gate="G$1" pin="8"/>
-<label x="40.64" y="17.78" size="1.778" layer="95"/>
+<wire x1="66.04" y1="17.78" x2="73.66" y2="17.78" width="0.1524" layer="91"/>
+<label x="66.04" y="17.78" size="1.778" layer="95"/>
 </segment>
 </net>
