File: avoccado-felina/avoccado-avr-pcb-felina.brd (EAGLE design)
At the start: 42.5 x 17.5 mm, 81 parts, among them Q1 16MHz, Q2 FET, U1 MPU-6000QFN-24, U2 MCP73831

Commit message: fix DRC errors
Parts:
- moved Q2 0.13 mm to (51.4, 15.2)
Routing:
- net GND: track 228.4 -> 227.8 mm
