File: avoccado-felina/avoccado-avr-pcb-felina-screwholes.sch (EAGLE design)
At the start: 81 parts, among them Q1 16MHz, Q2 FET, U1 MPU-6000QFN-24, U2 MCP73831

Commit message: add Felina fork with screw holes
Parts:
- C10: device rcl:C-EUC0402K -> rcl:C-EUC0603
Changed lines of the file:
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@@
 </classes>
 <parts>
-<part name="C10" library="rcl" deviceset="C-EU" device="C0402K" value="0.1uF"/>
+<part name="C10" library="rcl" deviceset="C-EU" device="C0603" value="0.1uF"/>
 <part name="FRAME1" library="SparkFun" deviceset="FRAME-LETTER" device=""/>
 <part name="GND25" library="SparkFun" deviceset="GND" device=""/>

Commit message: render schematic PNG
Other:
- note added: "CC-BY-SA 4.0 Avoccado° Creative Commons ShareAlike 4.0 International https://creativecommons.org/licenses/by-sa/4.0/ contact@avoccado.cc http://avoccado.cc"
- note added: "Main controller"
- note added: "peripheral connections"
- note removed: "main controller"
- note removed: "radio and MEMS connections"
Changed lines of the file:
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@@
 <text x="81.28" y="386.08" size="1.778" layer="91">R13, R14, R15 optional for v-usb mode. note: D2 also used at MPU6050</text>
 <text x="149.86" y="251.46" size="6.4516" layer="97" ratio="6">Power distribution</text>
-<text x="149.86" y="25.4" size="6.4516" layer="97" ratio="6">main controller</text>
+<text x="149.86" y="25.4" size="6.4516" layer="97" ratio="6">Main controller</text>
 <text x="439.42" y="25.4" size="6.4516" layer="97" ratio="6">TP and headers</text>
-<text x="723.9" y="25.4" size="6.4516" layer="97" ratio="6">radio and MEMS connections</text>
+<text x="723.9" y="25.4" size="6.4516" layer="97" ratio="6">peripheral connections</text>
 <text x="723.9" y="251.46" size="6.4516" layer="97" ratio="6">misc</text>
 <text x="439.42" y="251.46" size="6.4516" layer="97" ratio="6">MEMS</text>
@@
 <text x="175.26" y="381" size="1.778" layer="98">R3 determines the maximum charge current, 2K for 500 mA</text>
 <text x="609.6" y="251.46" size="1.778" layer="98">Fiducials 1 mm round</text>
+<text x="614.68" y="304.8" size="6.4516" layer="97">CC-BY-SA 4.0 Avoccado°
+Creative Commons ShareAlike 4.0 International
+https://creativecommons.org/licenses/by-sa/4.0/
+contact@avoccado.cc
+http://avoccado.cc</text>
 </plain>
 <instances>
@@
 </schematic>
 </drawing>
+<compatibility>
+<note version="6.3" minversion="6.2.2" severity="warning">
+Since Version 6.2.2 text objects can contain more than one line,
+which will not be processed correctly with this version.
+</note>
+</compatibility>
 </eagle>

Commit message: new footprint for USB
Parts:
- removed JP7: USB-MICROB, SparkFun-Connectors:USB-MICROB
- added JP22: USB_MICROB_PLUGCONN-11752, SparkFun-Connectors:USB_MICROB_PLUGCONN-11752
Connections:
- net 5V: now also JP22.VCC; no longer JP7.VBUS
- net GND: now also JP22.GND, JP22.SHIELD; no longer JP7.GND
- net N$4: now also JP22.D+; no longer JP7.D+
- net N$5: now also JP22.D-; no longer JP7.D-
Changed lines of the file:
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@@
 <part name="GND10" library="SparkFun" deviceset="GND" device=""/>
 <part name="MCU" library="SparkFun-DigitalIC" deviceset="ATMEGA328P_TQFP" device="" value="ATMEGA328P_TQFP"/>
-<part name="JP7" library="SparkFun-Connectors" deviceset="USB" device="-MICROB"/>
 <part name="R12" library="rcl" deviceset="R-EU_" device="R0402" value="1K"/>
 <part name="R9" library="rcl" deviceset="R-EU_" device="R0402" value="1K"/>
@@
 <part name="FID3" library="SparkFun-Aesthetics" deviceset="FIDUCIAL" device="UFIDUCIAL"/>
 <part name="FID4" library="SparkFun-Aesthetics" deviceset="FIDUCIAL" device="UFIDUCIAL"/>
+<part name="JP22" library="SparkFun-Connectors" deviceset="USB_MICROB_PLUG" device="CONN-11752"/>
+<part name="GND16" library="SparkFun" deviceset="GND" device=""/>
 </parts>
 <sheets>
@@
 <instance part="GND10" gate="1" x="17.78" y="314.96"/>
 <instance part="MCU" gate="U$1" x="193.04" y="124.46"/>
-<instance part="JP7" gate="G$1" x="86.36" y="365.76" rot="R180"/>
 <instance part="R12" gate="G$1" x="236.22" y="360.68" rot="R90"/>
 <instance part="R9" gate="G$1" x="236.22" y="347.98" rot="R90"/>
@@
 <instance part="FID3" gate="G$1" x="627.38" y="246.38"/>
 <instance part="FID4" gate="G$1" x="635" y="246.38"/>
+<instance part="JP22" gate="G$1" x="55.88" y="360.68" rot="R180"/>
+<instance part="GND16" gate="1" x="43.18" y="353.06"/>
 </instances>
 <busses>
@@
 <pinref part="GND8" gate="1" pin="GND"/>
 <wire x1="175.26" y1="353.06" x2="175.26" y2="347.98" width="0.1524" layer="91"/>
-<pinref part="JP7" gate="G$1" pin="GND"/>
 <wire x1="175.26" y1="347.98" x2="175.26" y2="330.2" width="0.1524" layer="91"/>
-<wire x1="88.9" y1="365.76" x2="142.24" y2="365.76" width="0.1524" layer="91"/>
+<wire x1="63.5" y1="365.76" x2="142.24" y2="365.76" width="0.1524" layer="91"/>
 <wire x1="142.24" y1="365.76" x2="142.24" y2="347.98" width="0.1524" layer="91"/>
 <wire x1="142.24" y1="347.98" x2="175.26" y2="347.98" width="0.1524" layer="91"/>
 <junction x="175.26" y="347.98"/>
+<pinref part="JP22" gate="G$1" pin="GND"/>
 </segment>
 <segment>
@@
 <wire x1="464.82" y1="58.42" x2="464.82" y2="88.9" width="0.1524" layer="91"/>
 <pinref part="TP4" gate="G$1" pin="TP"/>
+</segment>
+<segment>
+<pinref part="JP22" gate="G$1" pin="SHIELD"/>
+<pinref part="GND16" gate="1" pin="GND"/>
+<wire x1="48.26" y1="360.68" x2="43.18" y2="360.68" width="0.1524" layer="91"/>
+<wire x1="43.18" y1="360.68" x2="43.18" y2="355.6" width="0.1524" layer="91"/>
 </segment>
 </net>
@@
 <wire x1="175.26" y1="363.22" x2="175.26" y2="360.68" width="0.1524" layer="91"/>
 <label x="175.26" y="370.84" size="1.778" layer="95"/>
-<pinref part="JP7" gate="G$1" pin="VBUS"/>
-<wire x1="88.9" y1="363.22" x2="175.26" y2="363.22" width="0.1524" layer="91"/>
 <junction x="175.26" y="363.22"/>
+<wire x1="76.2" y1="363.22" x2="175.26" y2="363.22" width="0.1524" layer="91"/>
+<wire x1="76.2" y1="363.22" x2="76.2" y2="355.6" width="0.1524" layer="91"/>
+<pinref part="JP22" gate="G$1" pin="VCC"/>
+<wire x1="76.2" y1="355.6" x2="63.5" y2="355.6" width="0.1524" layer="91"/>
 </segment>
 <segment>
@@
 <net name="N$4" class="0">
 <segment>
-<pinref part="JP7" gate="G$1" pin="D+"/>
 <pinref part="R13" gate="G$1" pin="2"/>
-<wire x1="88.9" y1="358.14" x2="99.06" y2="358.14" width="0.1524" layer="91"/>
 <wire x1="99.06" y1="358.14" x2="99.06" y2="345.44" width="0.1524" layer="91"/>
+<wire x1="99.06" y1="358.14" x2="73.66" y2="358.14" width="0.1524" layer="91"/>
+<wire x1="73.66" y1="358.14" x2="73.66" y2="363.22" width="0.1524" layer="91"/>
+<wire x1="73.66" y1="363.22" x2="68.58" y2="363.22" width="0.1524" layer="91"/>
+<wire x1="68.58" y1="363.22" x2="68.58" y2="360.68" width="0.1524" layer="91"/>
+<pinref part="JP22" gate="G$1" pin="D+"/>
+<wire x1="68.58" y1="360.68" x2="63.5" y2="360.68" width="0.1524" layer="91"/>
 </segment>
 </net>
 <net name="N$5" class="0">
 <segment>
-<pinref part="JP7" gate="G$1" pin="D-"/>
 <pinref part="R14" gate="G$1" pin="2"/>
-<wire x1="88.9" y1="360.68" x2="109.22" y2="360.68" width="0.1524" layer="91"/>
+<wire x1="71.12" y1="360.68" x2="109.22" y2="360.68" width="0.1524" layer="91"/>
 <wire x1="109.22" y1="360.68" x2="109.22" y2="345.44" width="0.1524" layer="91"/>
-</segment>
-</net>
+<wire x1="71.12" y1="360.68" x2="71.12" y2="358.14" width="0.1524" layer="91"/>
+<pinref part="JP22" gate="G$1" pin="D-"/>
+<wire x1="71.12" y1="358.14" x2="63.5" y2="358.14" width="0.1524" layer="91"/>
+</segment>
+</net>

Commit message: eliminated redundant 0402 Rs for Rp
Parts:
- removed R12, R9: 1K, rcl:R-EU_R0402
Connections:
- removed net N$3: R12.1, R9.2
- net CHG-PROG: no longer R12.2
- net GND: no longer R9.1
Changed lines of the file:
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@@
 <part name="GND10" library="SparkFun" deviceset="GND" device=""/>
 <part name="MCU" library="SparkFun-DigitalIC" deviceset="ATMEGA328P_TQFP" device="" value="ATMEGA328P_TQFP"/>
-<part name="R12" library="rcl" deviceset="R-EU_" device="R0402" value="1K"/>
-<part name="R9" library="rcl" deviceset="R-EU_" device="R0402" value="1K"/>
 <part name="TP5" library="SparkFun-Passives" deviceset="TEST-POINT" device="3X5"/>
 <part name="TP3" library="SparkFun-Passives" deviceset="TEST-POINT" device="3X5"/>
@@
 <instance part="GND10" gate="1" x="17.78" y="314.96"/>
 <instance part="MCU" gate="U$1" x="193.04" y="124.46"/>
-<instance part="R12" gate="G$1" x="236.22" y="360.68" rot="R90"/>
-<instance part="R9" gate="G$1" x="236.22" y="347.98" rot="R90"/>
 <instance part="TP5" gate="G$1" x="114.3" y="279.4"/>
 <instance part="TP3" gate="G$1" x="114.3" y="263.144"/>
@@
 <pinref part="R3" gate="G$1" pin="1"/>
 <pinref part="GND3" gate="1" pin="GND"/>
-<wire x1="226.06" y1="355.6" x2="226.06" y2="337.82" width="0.1524" layer="91"/>
-<pinref part="R9" gate="G$1" pin="1"/>
-<wire x1="226.06" y1="337.82" x2="226.06" y2="330.2" width="0.1524" layer="91"/>
-<wire x1="236.22" y1="342.9" x2="236.22" y2="337.82" width="0.1524" layer="91"/>
-<wire x1="236.22" y1="337.82" x2="226.06" y2="337.82" width="0.1524" layer="91"/>
-<junction x="226.06" y="337.82"/>
+<wire x1="226.06" y1="355.6" x2="226.06" y2="330.2" width="0.1524" layer="91"/>
 </segment>
 <segment>
@@
 <pinref part="U2" gate="G$1" pin="PROG"/>
 <wire x1="226.06" y1="368.3" x2="213.36" y2="368.3" width="0.1524" layer="91"/>
-<pinref part="R12" gate="G$1" pin="2"/>
-<wire x1="226.06" y1="368.3" x2="236.22" y2="368.3" width="0.1524" layer="91"/>
-<wire x1="236.22" y1="368.3" x2="236.22" y2="365.76" width="0.1524" layer="91"/>
-<junction x="226.06" y="368.3"/>
 </segment>
 </net>
@@
 </segment>
 </net>
-<net name="N$3" class="0">
-<segment>
-<pinref part="R12" gate="G$1" pin="1"/>
-<pinref part="R9" gate="G$1" pin="2"/>
-<wire x1="236.22" y1="355.6" x2="236.22" y2="353.06" width="0.1524" layer="91"/>
-</segment>
-</net>

Commit message: no airwires left, added 5V USB power LED
Parts:
- removed TP14: TPTP20R, testpad:TPTP20R
- added D2: LED, SparkFun:LED0603
- added R9: 2K, rcl:R-EU_R0402
Connections:
- new net N$3: D2.A, R9.1
- net 5V: now also R9.2; no longer TP14.TP
- net GND: now also D2.C
Other:
- moved on the sheet: C4
Changed lines of the file:
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@@
 <part name="TP12" library="testpad" deviceset="TP" device="TP20R"/>
 <part name="TP13" library="testpad" deviceset="TP" device="TP20R"/>
-<part name="TP14" library="testpad" deviceset="TP" device="TP20R"/>
 <part name="TP4" library="testpad" deviceset="TP" device="TP20R"/>
 <part name="FRAME2" library="frames" deviceset="LETTER_L" device=""/>
@@
 <part name="JP22" library="SparkFun-Connectors" deviceset="USB_MICROB_PLUG" device="CONN-11752"/>
 <part name="GND16" library="SparkFun" deviceset="GND" device=""/>
+<part name="D2" library="SparkFun" deviceset="LED" device="0603" value="LED"/>
+<part name="GND17" library="SparkFun" deviceset="GND" device=""/>
+<part name="R9" library="rcl" deviceset="R-EU_" device="R0402" value="2K"/>
 </parts>
 <sheets>
@@
 <instance part="GND3" gate="1" x="226.06" y="327.66"/>
 <instance part="D1" gate="G$1" x="190.5" y="342.9" rot="MR0"/>
-<instance part="C4" gate="G$1" x="175.26" y="355.6"/>
+<instance part="C4" gate="G$1" x="167.64" y="355.6"/>
 <instance part="R4" gate="G$1" x="190.5" y="355.6" rot="R90"/>
 <instance part="GND6" gate="1" x="190.5" y="327.66"/>
-<instance part="GND8" gate="1" x="175.26" y="327.66"/>
+<instance part="GND8" gate="1" x="167.64" y="327.66"/>
 <instance part="GND9" gate="1" x="55.88" y="63.5"/>
 <instance part="R5" gate="G$1" x="45.72" y="76.2" rot="R90"/>
@@
 <instance part="TP12" gate="G$1" x="414.02" y="58.42" rot="R180"/>
 <instance part="TP13" gate="G$1" x="480.06" y="55.88" rot="R180"/>
-<instance part="TP14" gate="G$1" x="472.44" y="55.88" rot="R180"/>
 <instance part="TP4" gate="G$1" x="464.82" y="55.88" rot="R180"/>
 <instance part="FRAME2" gate="G$1" x="0" y="226.06"/>
@@
 <instance part="JP22" gate="G$1" x="55.88" y="360.68" rot="R180"/>
 <instance part="GND16" gate="1" x="43.18" y="353.06"/>
+<instance part="D2" gate="G$1" x="180.34" y="342.9" rot="MR0"/>
+<instance part="GND17" gate="1" x="180.34" y="327.66"/>
+<instance part="R9" gate="G$1" x="180.34" y="355.6" rot="R90"/>
 </instances>
 <busses>
@@
 <pinref part="C4" gate="G$1" pin="2"/>
 <pinref part="GND8" gate="1" pin="GND"/>
-<wire x1="175.26" y1="353.06" x2="175.26" y2="347.98" width="0.1524" layer="91"/>
-<wire x1="175.26" y1="347.98" x2="175.26" y2="330.2" width="0.1524" layer="91"/>
+<wire x1="167.64" y1="353.06" x2="167.64" y2="347.98" width="0.1524" layer="91"/>
+<wire x1="167.64" y1="347.98" x2="167.64" y2="330.2" width="0.1524" layer="91"/>
 <wire x1="63.5" y1="365.76" x2="142.24" y2="365.76" width="0.1524" layer="91"/>
 <wire x1="142.24" y1="365.76" x2="142.24" y2="347.98" width="0.1524" layer="91"/>
-<wire x1="142.24" y1="347.98" x2="175.26" y2="347.98" width="0.1524" layer="91"/>
-<junction x="175.26" y="347.98"/>
+<wire x1="142.24" y1="347.98" x2="167.64" y2="347.98" width="0.1524" layer="91"/>
+<junction x="167.64" y="347.98"/>
 <pinref part="JP22" gate="G$1" pin="GND"/>
 </segment>
@@
 <wire x1="48.26" y1="360.68" x2="43.18" y2="360.68" width="0.1524" layer="91"/>
 <wire x1="43.18" y1="360.68" x2="43.18" y2="355.6" width="0.1524" layer="91"/>
+</segment>
+<segment>
+<pinref part="D2" gate="G$1" pin="C"/>
+<pinref part="GND17" gate="1" pin="GND"/>
+<wire x1="180.34" y1="337.82" x2="180.34" y2="330.2" width="0.1524" layer="91"/>
 </segment>
 </net>
@@
 <segment>
 <pinref part="U2" gate="G$1" pin="VIN"/>
-<wire x1="175.26" y1="363.22" x2="175.26" y2="370.84" width="0.1524" layer="91"/>
-<wire x1="175.26" y1="370.84" x2="193.04" y2="370.84" width="0.1524" layer="91"/>
+<wire x1="167.64" y1="363.22" x2="167.64" y2="370.84" width="0.1524" layer="91"/>
 <pinref part="C4" gate="G$1" pin="1"/>
-<wire x1="175.26" y1="363.22" x2="175.26" y2="360.68" width="0.1524" layer="91"/>
-<label x="175.26" y="370.84" size="1.778" layer="95"/>
-<junction x="175.26" y="363.22"/>
-<wire x1="76.2" y1="363.22" x2="175.26" y2="363.22" width="0.1524" layer="91"/>
+<wire x1="167.64" y1="370.84" x2="180.34" y2="370.84" width="0.1524" layer="91"/>
+<wire x1="180.34" y1="370.84" x2="193.04" y2="370.84" width="0.1524" layer="91"/>
+<wire x1="167.64" y1="363.22" x2="167.64" y2="360.68" width="0.1524" layer="91"/>
+<label x="167.64" y="370.84" size="1.778" layer="95"/>
+<junction x="167.64" y="363.22"/>
+<wire x1="76.2" y1="363.22" x2="167.64" y2="363.22" width="0.1524" layer="91"/>
 <wire x1="76.2" y1="363.22" x2="76.2" y2="355.6" width="0.1524" layer="91"/>
 <pinref part="JP22" gate="G$1" pin="VCC"/>
 <wire x1="76.2" y1="355.6" x2="63.5" y2="355.6" width="0.1524" layer="91"/>
+<pinref part="R9" gate="G$1" pin="2"/>
+<wire x1="180.34" y1="360.68" x2="180.34" y2="370.84" width="0.1524" layer="91"/>
+<junction x="180.34" y="370.84"/>
 </segment>
 <segment>
@@
 <pinref part="JP17" gate="G$1" pin="1"/>
 <label x="495.3" y="124.46" size="1.778" layer="95"/>
-</segment>
-<segment>
-<wire x1="472.44" y1="88.9" x2="472.44" y2="58.42" width="0.1524" layer="91"/>
-<pinref part="TP14" gate="G$1" pin="TP"/>
-<label x="472.44" y="88.9" size="1.778" layer="95" rot="R270"/>
 </segment>
 </net>
@@
 </segment>
 </net>
+<net name="N$3" class="0">
+<segment>
+<pinref part="D2" gate="G$1" pin="A"/>
+<pinref part="R9" gate="G$1" pin="1"/>
+<wire x1="180.34" y1="345.44" x2="180.34" y2="350.52" width="0.1524" layer="91"/>
+</segment>
+</net>

Commit message: add redundant fiducials near mounting holes, reverse LED and R
Parts:
- added FID5, FID6, FID7, FID8, FID9: FIDUCIALUFIDUCIAL, SparkFun-Aesthetics:FIDUCIALUFIDUCIAL
Connections:
- net 5V: now also D2.A; no longer R9.2
- net GND: now also R9.1; no longer D2.C
- net N$3: now also D2.C, R9.2; no longer D2.A, R9.1
Other:
- moved on the sheet: D2, R9
Changed lines of the file:
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@@
 <part name="FID1" library="SparkFun-Aesthetics" deviceset="FIDUCIAL" device="UFIDUCIAL"/>
 <part name="FID3" library="SparkFun-Aesthetics" deviceset="FIDUCIAL" device="UFIDUCIAL"/>
-<part name="FID4" library="SparkFun-Aesthetics" deviceset="FIDUCIAL" device="UFIDUCIAL"/>
 <part name="JP22" library="SparkFun-Connectors" deviceset="USB_MICROB_PLUG" device="CONN-11752"/>
 <part name="GND16" library="SparkFun" deviceset="GND" device=""/>
@@
 <part name="GND17" library="SparkFun" deviceset="GND" device=""/>
 <part name="R9" library="rcl" deviceset="R-EU_" device="R0402" value="2K"/>
+<part name="FID4" library="SparkFun-Aesthetics" deviceset="FIDUCIAL" device="UFIDUCIAL"/>
+<part name="FID5" library="SparkFun-Aesthetics" deviceset="FIDUCIAL" device="UFIDUCIAL"/>
+<part name="FID6" library="SparkFun-Aesthetics" deviceset="FIDUCIAL" device="UFIDUCIAL"/>
+<part name="FID7" library="SparkFun-Aesthetics" deviceset="FIDUCIAL" device="UFIDUCIAL"/>
+<part name="FID8" library="SparkFun-Aesthetics" deviceset="FIDUCIAL" device="UFIDUCIAL"/>
+<part name="FID9" library="SparkFun-Aesthetics" deviceset="FIDUCIAL" device="UFIDUCIAL"/>
 </parts>
 <sheets>
@@
 <instance part="FID1" gate="G$1" x="619.76" y="246.38"/>
 <instance part="FID3" gate="G$1" x="627.38" y="246.38"/>
-<instance part="FID4" gate="G$1" x="635" y="246.38"/>
 <instance part="JP22" gate="G$1" x="55.88" y="360.68" rot="R180"/>
 <instance part="GND16" gate="1" x="43.18" y="353.06"/>
-<instance part="D2" gate="G$1" x="180.34" y="342.9" rot="MR0"/>
-<instance part="GND17" gate="1" x="180.34" y="327.66"/>
-<instance part="R9" gate="G$1" x="180.34" y="355.6" rot="R90"/>
+<instance part="D2" gate="G$1" x="180.34" y="368.3" rot="MR0"/>
+<instance part="GND17" gate="1" x="180.34" y="314.96"/>
+<instance part="R9" gate="G$1" x="180.34" y="327.66" rot="R90"/>
+<instance part="FID4" gate="G$1" x="635" y="246.38"/>
+<instance part="FID5" gate="G$1" x="642.62" y="246.38"/>
+<instance part="FID6" gate="G$1" x="612.14" y="241.3"/>
+<instance part="FID7" gate="G$1" x="619.76" y="241.3"/>
+<instance part="FID8" gate="G$1" x="627.38" y="241.3"/>
+<instance part="FID9" gate="G$1" x="635" y="241.3"/>
 </instances>
 <busses>
@@
 </segment>
 <segment>
-<pinref part="D2" gate="G$1" pin="C"/>
 <pinref part="GND17" gate="1" pin="GND"/>
-<wire x1="180.34" y1="337.82" x2="180.34" y2="330.2" width="0.1524" layer="91"/>
+<pinref part="R9" gate="G$1" pin="1"/>
+<wire x1="180.34" y1="317.5" x2="180.34" y2="322.58" width="0.1524" layer="91"/>
 </segment>
 </net>
@@
 <pinref part="JP22" gate="G$1" pin="VCC"/>
 <wire x1="76.2" y1="355.6" x2="63.5" y2="355.6" width="0.1524" layer="91"/>
-<pinref part="R9" gate="G$1" pin="2"/>
-<wire x1="180.34" y1="360.68" x2="180.34" y2="370.84" width="0.1524" layer="91"/>
+<pinref part="D2" gate="G$1" pin="A"/>
 <junction x="180.34" y="370.84"/>
 </segment>
@@
 <net name="N$3" class="0">
 <segment>
-<pinref part="D2" gate="G$1" pin="A"/>
-<pinref part="R9" gate="G$1" pin="1"/>
-<wire x1="180.34" y1="345.44" x2="180.34" y2="350.52" width="0.1524" layer="91"/>
-</segment>
-</net>
+<pinref part="R9" gate="G$1" pin="2"/>
+<pinref part="D2" gate="G$1" pin="C"/>
+<wire x1="180.34" y1="363.22" x2="180.34" y2="332.74" width="0.1524" layer="91"/>
+</segment>
+</net>

Commit message: increase trace width for Vcc near edges
Other:
- note added: "NRF24L01+ board header SPI (IRQ at ADC7 / A7)"
- note removed: "NRF24L01+ board header SPI (IRQ at A7)"
- moved on the sheet: C1
Changed lines of the file:
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@@
 <sheet>
 <plain>
-<text x="650.24" y="96.52" size="1.778" layer="91" rot="R180">NRF24L01+ board header SPI (IRQ at A7)</text>
+<text x="650.24" y="96.52" size="1.778" layer="91" rot="R180">NRF24L01+ board header SPI (IRQ at ADC7 / A7)</text>
 <text x="741.68" y="99.06" size="1.778" layer="91" rot="R180">MPU6050 minimal header I2C</text>
 <text x="175.26" y="162.56" size="1.778" layer="91">AtMega 328p</text>
@@
 </instance>
 <instance part="GND1" gate="1" x="154.94" y="93.98"/>
-<instance part="C1" gate="G$1" x="149.86" y="134.62" smashed="yes" rot="R180">
-<attribute name="NAME" x="150.876" y="134.747" size="1.778" layer="95"/>
-<attribute name="VALUE" x="150.876" y="129.921" size="1.778" layer="96"/>
+<instance part="C1" gate="G$1" x="134.62" y="134.62" smashed="yes" rot="R180">
+<attribute name="NAME" x="135.636" y="134.747" size="1.778" layer="95"/>
+<attribute name="VALUE" x="135.636" y="129.921" size="1.778" layer="96"/>
 </instance>
-<instance part="GND7" gate="1" x="149.86" y="124.46"/>
+<instance part="GND7" gate="1" x="134.62" y="124.46"/>
 <instance part="GND30" gate="1" x="63.5" y="248.92"/>
 <instance part="GND32" gate="1" x="40.64" y="248.92"/>
@@
 </segment>
 <segment>
-<wire x1="149.86" y1="127" x2="149.86" y2="132.08" width="0.1524" layer="91"/>
+<wire x1="134.62" y1="127" x2="134.62" y2="132.08" width="0.1524" layer="91"/>
 <pinref part="C1" gate="G$1" pin="1"/>
 <pinref part="GND7" gate="1" pin="GND"/>
@@
 <wire x1="377.19" y1="148.844" x2="310.134" y2="148.844" width="0.1524" layer="91"/>
 <pinref part="JP5" gate="G$1" pin="1"/>
+<label x="377.19" y="148.844" size="1.778" layer="95"/>
 </segment>
 <segment>
@@
 <wire x1="464.82" y1="58.42" x2="464.82" y2="88.9" width="0.1524" layer="91"/>
 <pinref part="TP4" gate="G$1" pin="TP"/>
+<label x="464.82" y="88.9" size="1.778" layer="95" rot="R270"/>
 </segment>
 <segment>
@@
 <net name="AREF" class="0">
 <segment>
-<wire x1="167.64" y1="139.7" x2="149.86" y2="139.7" width="0.1524" layer="91"/>
+<wire x1="167.64" y1="139.7" x2="134.62" y2="139.7" width="0.1524" layer="91"/>
 <label x="157.48" y="139.7" size="1.778" layer="95"/>
 <pinref part="C1" gate="G$1" pin="2"/>
@@
 <wire x1="377.19" y1="151.638" x2="321.31" y2="151.638" width="0.1524" layer="91"/>
 <pinref part="JP4" gate="G$1" pin="1"/>
-</segment>
-<segment>
+<label x="377.444" y="151.892" size="1.778" layer="95"/>
+</segment>
+<segment>
