File: avoccado-gin/panel/avoccado-avr-gin-panel.sch (EAGLE design)
At the start: 83 parts, among them Q1 16MHz, Q2 FET, U1 MPU-6000QFN-24, U2 MCP73831

Commit message: Felina: remove screw mounts, Gin: prepare to panelize
Parts:
- removed D2: LED, SparkFun:LED0603
- removed FID7: FIDUCIALUFIDUCIAL, SparkFun-Aesthetics:FIDUCIALUFIDUCIAL
- removed JP1, JP12, JP14, JP15, JP16, JP20, JP30, JP31, JP4, JP5: M01NOSILK-KIT, SparkFun-Connectors:M01NOSILK-KIT
- removed JP10, JP11, JP13, JP17, JP18, JP19, JP21, JP23, JP24, JP25, JP3, JP6, JP8, JP9: M01PTH, SparkFun-Connectors:M01PTH
- removed LOGO1: OSHW-LOGOS, SparkFun-Aesthetics:OSHW-LOGOS
- removed MCU: ATMEGA328P_TQFP, SparkFun-DigitalIC:ATMEGA328P_TQFP
- removed R13, R14: 68R, SparkFun-Resistors:RESISTOR0603
- removed R15: 2K, SparkFun-Resistors:RESISTOR0603
- removed R9: 2K, rcl:R-EU_R0402
- removed TP13: TPTP20R, testpad:TPTP20R
- added FID4, FID6: FIDUCIALUFIDUCIAL, SparkFun-Aesthetics:FIDUCIALUFIDUCIAL
- added TP14, TP15, TP16, TP17: TPTP20R, testpad:TPTP20R
- added U3: (no value), SparkFun-DigitalIC:ATMEGA328P_MLFMLF32
- C10: value 0.1uF -> 4.7uF
- C2: device rcl:C-EUC0402K -> resistor:C-EUC0402K
- Q2: value FET -> N-FET
- TP1, TP11, TP6, TP7, TP8, TP9: value TEST-POINT2 -> TPTP20R; device SparkFun-Passives:TEST-POINT2 -> testpad:TPTP20R
- TP2: value M01PTH -> TPTP20R; device SparkFun-Connectors:M01PTH -> testpad:TPTP20R
Connections:
- removed net 7-TO-D-: R14.1, R15.1, TP11.1
- removed net DTR: C2.2, JP10.1
- removed net N$3: D2.C, R9.2
- removed net N$4: JP22.D+, R13.2
- removed net N$5: JP22.D-, R14.2
- net 3.3V: now also C2.2, TP9.TP, U3.AVCC, U3.VCC@4, U3.VCC@6; no longer JP1.1, JP11.1, JP18.1, JP4.1, MCU.AVCC, MCU.VCC@4, MCU.VCC@6, R15.2, TP13.TP
- net 5V: no longer D2.A, JP17.1
- net A0: now also U3.PC0(ADC0); no longer JP19.1, MCU.PC0(ADC0)
- net A1: now also TP8.TP, U3.PC1(ADC1); no longer JP20.1, MCU.PC1(ADC1)
- net A2: now also U3.PC2(ADC2); no longer JP21.1, MCU.PC2(ADC2)
- net A3: now also U3.PC3(ADC3); no longer MCU.PC3(ADC3)
- net A4: now also U3.PC4(ADC4/SDA); no longer JP31.1, MCU.PC4(ADC4/SDA)
- net A5: now also U3.PC5(ADC5/SCL); no longer JP30.1, MCU.PC5(ADC5/SCL)
- net A6: now also U3.ADC6; no longer MCU.ADC6
- net A7-NRF-IRQ: now also U3.ADC7; no longer JP29.2, MCU.ADC7
- net AREF: now also U3.AREF; no longer MCU.AREF
- net D10: now also U3.PB2(SS/OC1B); no longer MCU.PB2(SS/OC1B)
- net D2-INT: now also U3.PD2(INT0); no longer MCU.PD2(INT0), R13.1, TP2.1
- net D3: now also U3.PD3(INT1); no longer MCU.PD3(INT1)
- net D4: now also U3.PD4(XCK/T0); no longer MCU.PD4(XCK/T0)
- net D5: now also TP15.TP, U3.PD5(T1); no longer MCU.PD5(T1), TP1.1
- net D6: now also U3.PD6(AIN0); no longer MCU.PD6(AIN0), TP6.1
- net D7: now also TP14.TP, U3.PD7(AIN1); no longer MCU.PD7(AIN1), TP7.1
- net D8: now also TP11.TP, U3.PB0(ICP); no longer MCU.PB0(ICP), TP8.1
- net D9: now also U3.PB1(OC1A); no longer MCU.PB1(OC1A)
- net GND: now also C2.1, TP16.TP, TP17.TP, U3.AGND, U3.GND@3, U3.GND@5, U3.GND@PAD; no longer JP16.1, JP25.1, JP3.1, JP5.1, JP6.1, MCU.AGND, MCU.GND@3, MCU.GND@5, R9.1, TP4.TP, TP9.1
- net MISO: now also U3.PB4(MISO); no longer JP12.1, MCU.PB4(MISO)
- net MOSI: now also U3.PB3(MOSI/OC2); no longer JP14.1, MCU.PB3(MOSI/OC2)
- net N$1: now also U3.PB7(XTAL2/TOSC2); no longer MCU.PB7(XTAL2/TOSC2)
- net N$2: now also U3.PB6(XTAL1/TOSC1); no longer MCU.PB6(XTAL1/TOSC1)
- net RESET: now also TP7.TP, U3.PC6(/RESET); no longer C2.1, JP15.1, MCU.PC6(/RESET)
- net RXI: now also TP2.TP, U3.PD0(RXD); no longer JP8.1, MCU.PD0(RXD)
- net SCK: now also U3.PB5(SCK); no longer JP13.1, MCU.PB5(SCK)
- net TXO: now also TP6.TP, U3.PD1(TXD); no longer JP9.1, MCU.PD1(TXD)
- net VBAT: now also TP4.TP; no longer JP24.1
- net VIBR: now also TP1.TP; no longer JP23.1
Other:
- note added: "NRF24L01+ board header SPI (IRQ NC)"
- note removed: "ICSP header"
- note removed: "MPU6050 minimal header I2C"
- note removed: "NRF24L01+ board header SPI (IRQ at ADC7 / A7)"
- note removed: "Needs to be bridged to D7 with an air wire for v-usb"
- note removed: "Optional for v-usb"
- moved on the sheet: C2
