File: avoccado-panel-felina-faye-gin/avoccado-panel-felina-faye-gin.brd (EAGLE design)
At the start: 100.5 x 100.5 mm, 852 parts, among them Q1 16MHz, Q10 FET, Q11 16MHz, Q12 FET, Q13 16MHz, Q14 N-FET, Q15 16MHz, Q16 N-FET, Q17 16MHz, Q18 FET, Q19 16MHz, Q2 FET, Q20 FET, Q21 16MHz, Q22 FET, Q23 16MHz, Q24 FET, Q3 16MHz, Q4 FET, Q5 16MHz, Q6 FET, Q7 16MHz, Q8 FET, Q9 16MHz, U1 MPU-6000QFN-24, U10 MPU-6000QFN-24, U11 MCP73831, U12 MPU-6000QFN-24, U13 MCP73831, U14 MPU-6000QFN-24, U16 MCP73831, U17 MPU-6000QFN-24, U19 MCP73831, U2 MCP73831, U22 MCP73831, U23 MCP73831, U24 MCP73831, U3 MCP73831, U4 MPU-6000QFN-24, U5 MCP73831, U6 MPU-6000QFN-24, U7 MCP73831, U8 MPU-6000QFN-24, U9 MCP73831

Commit message: add PCBs with ICSP adapters and panelize
Parts:
- added C124, C125, C126: 4.7uF, SparkFun-Capacitors:0603-CAP
- added C127, C128, C130: 0.1uF, rcl:C0402K
- added C129: 2.2nF, rcl:C0402K
- added C131, C98, C99: 0.1uF, resistor:C0402K
- added C132: (no value), rcl:C0402
- added C97: 4.7uF, rcl:C0603
- added D19: LED, SparkFun:LED-0603
- added FID55, FID56, FID57, FID58, FID59, FID60: FIDUCIALUFIDUCIAL, SparkFun-Aesthetics:MICRO-FIDUCIAL
- added JP293, JP294, JP295, JP296, JP876, JP877, JP878, JP879: M021X02_NO_SILK, SparkFun-Connectors:1X02_NO_SILK
- added JP297: USB_MICROB_PLUGCONN-11752, SparkFun-Connectors:USB-B-MICRO-SMD_V03
- added LDO12: MCP1703CB, linear:SOT23
- added Q25: 16MHz, SparkFun:RESONATOR-SMD
- added Q26: N-FET, SparkFun-DiscreteSemi:SOT23-3
- added R145, R153, R154: 10K, SparkFun-Resistors:0603-RES
- added R146, R150: 511R, SparkFun-Resistors:0603-RES
- added R147, R148: 2K, SparkFun-Resistors:0603-RES
- added R149, R151, R152: 4.7M, SparkFun-Resistors:0603-RES
- added TP120, TP121: TEST-POINT3X5, SparkFun-Passives:PAD.03X.05
- added TP122, TP123, TP124, TP125, TP126, TP154, TP155, TP156, TP157, TP158, TP159, TP160, TP161, TP162: TPTP20R, testpad:TP20R
- added TP163, TP164, TP165, TP166, TP167, TP168, TP169, TP170, TP171, TP172, TP173, TP174, TP175, TP176, TP177, TP178, TP179, TP180, TP181, TP559, TP560, TP561, TP562, TP563, TP564: PTR1PAD1-13, testpad:P1-13
- added U$1, U$6: AVR_SPI_PROG, SparkFun-Connectors:AVR_ICSP
- added U20: MCP73831, SparkFun:SOT23-5
- added U21: MPU-6000QFN-24, SparkFun-Sensors:QFN-24-TESTING
- added U25: (no value), SparkFun-DigitalIC:MLF32-PAD
- moved TP85 109.0 mm to (4.61, 59.6), turned to 0 degrees
- moved JP178 108.3 mm to (4.61, 62.1), turned to 0 degrees
- moved FID43 108.2 mm to (3.46, 70.9), turned to 0 degrees
- moved FID47 108.2 mm to (3.46, 70.9), turned to 0 degrees
- moved JP177 107.6 mm to (4.61, 64.7), turned to 0 degrees
- moved FID46 107.2 mm to (5.62, 60.7), turned to 0 degrees
- moved JP176 107.1 mm to (4.61, 67.2), turned to 0 degrees
- moved FID44 106.9 mm to (5.88, 60.6), turned to 0 degrees
- moved JP175 106.7 mm to (4.61, 69.8), turned to 0 degrees
- moved R91 105.5 mm to (7.15, 59.5), turned to 0 degrees
- moved TP86 105.5 mm to (7.15, 59.6), turned to 0 degrees
- moved TP81 102.0 mm to (9.69, 59.6), turned to 0 degrees
- moved C73 101.9 mm to (8.93, 63.4), turned to 90 degrees
- moved R92 101.8 mm to (9.69, 60.4), turned to 270 degrees
- moved C69 101.3 mm to (8.93, 65.8), turned to 90 degrees
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Connections:
- new net 3.3V12: C126.1, C131.2, C97.1, C98.2, JP293.2, LDO12.2, R145.2, R153.2, R154.2, TP120.P$1, TP157.TP, U21.13, U25.18, U25.4, U25.6
- new net 3.3V13: TP169.TP, TP175.TP, TP180.TP, U$1.2
- new net 3.3V44: JP876.2, TP560.TP, U$6.2
- new net 5V12: C124.1, JP297.VBUS1, U20.4
- new net A7-NRF-IRQ12: U25.22
- new net A7-NRF-IRQ41: JP879.2
- new net A84: R153.1, U21.23, U25.28
- new net A85: R154.1, U21.24, U25.27
- new net A86: C127.1, R151.2, R152.1, U25.26
- new net A87: U25.25
- new net A88: TP156.TP, U25.24
- new net A89: U25.23
- new net A90: U25.19
- new net AREF12: C99.2, U25.20
- new net CHG-PROG12: R147.2, U20.5
- new net D101: JP294.1, U25.13
- new net D102: TP158.TP, U25.12
- new net D103: R150.1, U25.1
- new net D104: R146.1, U25.2
- new net D105: TP160.TP, U25.9
- new net D106: U25.10
- new net D107: TP159.TP, U25.11
- new net D108: JP294.2, U25.14
- new net D109: TP164.TP
- new net D110: TP163.TP
- new net D111: TP165.TP
- new net D2-INT8: U21.12, U25.32
- new net D338: JP877.1
- new net D339: JP877.2
- new net DTR29: C132.2, TP172.TP
- new net GND12: C124.2, C125.2, C126.2, C127.2, C128.2, C129.2, C130.2, C131.1, C97.2, C98.1, C99.1, D19.C, JP293.1, JP297.GND1, JP297.SHIELD1, JP297.SHIELD2, JP297.SHIELD3, LDO12.1, Q25.2, Q26.2, R147.1, R149.1, R151.1, TP121.P$1, TP123.TP, TP161.TP, TP162.TP, U20.2, U21.1, U21.11, U21.18, U21.9, U25.21, U25.3, U25.5, U25.PAD
- new net GND13: TP170.TP, TP176.TP, TP181.TP, U$1.10
- new net GND44: JP876.1, TP559.TP, U$6.10
- new net LED12: D19.A, R148.1, R150.2
- new net MISO12: JP296.1, U25.16
- new net MISO13: TP179.TP, U$1.9
- new net MISO44: JP879.1, TP563.TP, U$6.9
- new net MOSI12: JP295.2, U25.15
- new net MOSI13: TP177.TP, U$1.1
- new net MOSI44: JP878.2, TP561.TP, U$6.1
- new net N$71: Q25.1, U25.8
- new net N$72: Q25.3, U25.7
- new net N$85: Q26.1, R146.2, R149.2
- new net N$86: C128.1, U21.10
- new net N$87: C129.1, U21.20
- new net N$88: C130.1, U21.8
- new net RESET12: R145.1, TP155.TP, U25.29
- new net RESET13: C132.1, TP166.TP, U$1.5
- new net RESET44: TP564.TP, U$6.5
- new net RXI12: TP126.TP, U25.30
- new net RXI13: TP167.TP, TP173.TP
- new net SCK12: JP295.1, U25.17
- new net SCK13: TP178.TP, U$1.7
- new net SCK44: JP878.1, TP562.TP, U$6.7
- new net SOC12: R148.2, U20.1
- new net TXO12: TP154.TP, U25.31
- new net TXO13: TP168.TP, TP174.TP
- new net VBAT12: C125.1, LDO12.3, R152.2, TP122.TP, TP124.TP, U20.3
- new net VBAT13: TP171.TP
- new net VIBR12: Q26.3, TP125.TP
Routing:
- net GND19: track 0.00 -> 212.0 mm, vias 0 -> 11
- net GND14: track 0.00 -> 212.0 mm, vias 0 -> 11
- net GND22: track 0.00 -> 212.0 mm, vias 0 -> 11
- net GND21: track 0.00 -> 212.0 mm, vias 0 -> 11
- net GND20: track 0.00 -> 212.0 mm, vias 0 -> 11
- net GND34: track 0.00 -> 212.0 mm, vias 0 -> 11
- net GND32: track 0.00 -> 212.0 mm, vias 0 -> 11
- net GND31: track 0.00 -> 212.0 mm, vias 0 -> 11
- net GND33: track 0.00 -> 212.0 mm, vias 0 -> 11
- net GND30: track 0.00 -> 212.0 mm, vias 0 -> 11
- net 3.3V22: track 0.00 -> 173.8 mm, vias 0 -> 4
- net 3.3V21: track 0.00 -> 173.8 mm, vias 0 -> 4
- net 3.3V20: track 0.00 -> 173.8 mm, vias 0 -> 4
- net 3.3V19: track 0.00 -> 173.8 mm, vias 0 -> 4
- net 3.3V14: track 0.00 -> 173.8 mm, vias 0 -> 4
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- added copper zone on layer 1, net GND12
- added copper zone on layer 16, net GND12
- added copper zone on layer 1, net GND13
- added copper zone on layer 16, net GND13
- added copper zone on layer 1, net GND14
- added copper zone on layer 1, net GND15
- added copper zone on layer 16, net GND15
- added copper zone on layer 1, net GND16
- added copper zone on layer 16, net GND16
- added copper zone on layer 1, net GND17
- added copper zone on layer 16, net GND17
- added copper zone on layer 1, net GND18
- added copper zone on layer 16, net GND18
- added copper zone on layer 1, net GND19
- added copper zone on layer 16, net GND19
- added copper zone on layer 1, net GND20
- added copper zone on layer 16, net GND20
- added copper zone on layer 1, net GND21
- added copper zone on layer 16, net GND21
- added copper zone on layer 1, net GND22
- added copper zone on layer 16, net GND22
- added copper zone on layer 1, net GND24
- added copper zone on layer 16, net GND24
- added copper zone on layer 1, net GND25
- added copper zone on layer 16, net GND25
- added copper zone on layer 1, net GND26
- added copper zone on layer 16, net GND26
- added copper zone on layer 1, net GND27
- added copper zone on layer 16, net GND27
- added copper zone on layer 1, net GND28
- added copper zone on layer 16, net GND28
- added copper zone on layer 1, net GND29
- added copper zone on layer 1, net GND30
- added copper zone on layer 16, net GND30
- added copper zone on layer 1, net GND31
- added copper zone on layer 16, net GND31
- added copper zone on layer 1, net GND32
- added copper zone on layer 16, net GND32
- added copper zone on layer 1, net GND33
- added copper zone on layer 16, net GND33
- added copper zone on layer 1, net GND34
- added copper zone on layer 16, net GND34
- added copper zone on layer 1, net GND35
- added copper zone on layer 16, net GND35
- added copper zone on layer 1, net GND36
- added copper zone on layer 16, net GND36
- added copper zone on layer 1, net GND37
- added copper zone on layer 16, net GND37
- added copper zone on layer 1, net GND38
- added copper zone on layer 16, net GND38
- added copper zone on layer 1, net GND44
- added copper zone on layer 16, net GND44
Other:
- board size 100.5 x 100.5 mm -> 100.5 x 101 mm
- board text added: "AVOCCADO.CC"
- board text added: "D T R V G"
- board text added: "FELINA ICSP"
- board text added: "LIBRE HARDWARE"
- board text added: "RST"
- board text added: "SHURE OPEN TECHNOLOGIES"
- board text removed: "OCC DO GIN"
